File: keyboard.kicad_sch (KiCad schematic)
At the start: 168 parts

Commit message: pico breakout version
Parts:
- removed L0: SK6812MINI, LED_SMD:LED_SK6812MINI_PLCC4_3.5x3.5mm_P1.75mm, symbol LED:SK6812MINI
- added D16: D, Diode_SMD:D_SOD-123, symbol Device:D
- added H1, H10, H2, H3, H4, H5, H6, H7, H8, H9: MountingHole, MountingHole:MountingHole_2.2mm_M2, symbol Mechanical:MountingHole
- added R1, R2: 4.7k, Resistor_SMD:R_0603_1608Metric, symbol Device:R
- added S16: Magic, keyboard:MX-Hotswap-1U, symbol keyswitch:Placeholder_Keyswitch
- added U1: OLED96-636, keyboard:MODULE_DM-OLED096-636, symbol extra_stuff:OLED_DISPLAY_I2C
- D1: renamed from D0; footprint (none) -> Diode_SMD:D_SOD-123
- D10: renamed from D9; footprint (none) -> Diode_SMD:D_SOD-123
- D11: renamed from D10; footprint (none) -> Diode_SMD:D_SOD-123
- D12: renamed from D11; footprint (none) -> Diode_SMD:D_SOD-123
- D13: renamed from D12; footprint (none) -> Diode_SMD:D_SOD-123
- D14: renamed from D13; footprint (none) -> Diode_SMD:D_SOD-123
- D15: renamed from D14; footprint (none) -> Diode_SMD:D_SOD-123
- D17: renamed from D15; footprint (none) -> Diode_SMD:D_SOD-123
- D18: renamed from D16; footprint (none) -> Diode_SMD:D_SOD-123
- D19: renamed from D17; footprint (none) -> Diode_SMD:D_SOD-123
- D2: renamed from D1; footprint (none) -> Diode_SMD:D_SOD-123
- D20: renamed from D18; footprint (none) -> Diode_SMD:D_SOD-123
- D21: renamed from D19; footprint (none) -> Diode_SMD:D_SOD-123
- D22: renamed from D20; footprint (none) -> Diode_SMD:D_SOD-123
- D23: renamed from D21; footprint (none) -> Diode_SMD:D_SOD-123
- D24: renamed from D22; footprint (none) -> Diode_SMD:D_SOD-123
- D25: renamed from D23; footprint (none) -> Diode_SMD:D_SOD-123
- D26: renamed from D24; footprint (none) -> Diode_SMD:D_SOD-123
- D27: renamed from D25; footprint (none) -> Diode_SMD:D_SOD-123
- D28: renamed from D26; footprint (none) -> Diode_SMD:D_SOD-123
- D29: renamed from D27; footprint (none) -> Diode_SMD:D_SOD-123
- D3: renamed from D2; footprint (none) -> Diode_SMD:D_SOD-123
- D30: renamed from D28; footprint (none) -> Diode_SMD:D_SOD-123
- D31: renamed from D29; footprint (none) -> Diode_SMD:D_SOD-123
- D32: renamed from D30; footprint (none) -> Diode_SMD:D_SOD-123
- D33: renamed from D31; footprint (none) -> Diode_SMD:D_SOD-123
- D34: renamed from D32; footprint (none) -> Diode_SMD:D_SOD-123
- D35: renamed from D33; footprint (none) -> Diode_SMD:D_SOD-123
- D36: renamed from D34; footprint (none) -> Diode_SMD:D_SOD-123
- D37: renamed from D35; footprint (none) -> Diode_SMD:D_SOD-123
- D38: renamed from D36; footprint (none) -> Diode_SMD:D_SOD-123
- D39: renamed from D37; footprint (none) -> Diode_SMD:D_SOD-123
- D4: renamed from D3; footprint (none) -> Diode_SMD:D_SOD-123
- D40: renamed from D38; footprint (none) -> Diode_SMD:D_SOD-123
- D41: renamed from D39; footprint (none) -> Diode_SMD:D_SOD-123
- D42: renamed from D40; footprint (none) -> Diode_SMD:D_SOD-123
- D43: renamed from D41; footprint (none) -> Diode_SMD:D_SOD-123
- D44: renamed from D42; footprint (none) -> Diode_SMD:D_SOD-123
- D45: renamed from D43; footprint (none) -> Diode_SMD:D_SOD-123
- D46: renamed from D44; footprint (none) -> Diode_SMD:D_SOD-123
- D47: renamed from D45; footprint (none) -> Diode_SMD:D_SOD-123
- D48: renamed from D46; footprint (none) -> Diode_SMD:D_SOD-123
- D49: renamed from D47; footprint (none) -> Diode_SMD:D_SOD-123
- D5: renamed from D4; footprint (none) -> Diode_SMD:D_SOD-123
- D50: renamed from D48; footprint (none) -> Diode_SMD:D_SOD-123
- D51: renamed from D49; footprint (none) -> Diode_SMD:D_SOD-123
- D52: renamed from D50; footprint (none) -> Diode_SMD:D_SOD-123
- D53: renamed from D51; footprint (none) -> Diode_SMD:D_SOD-123
- D54: renamed from D52; footprint (none) -> Diode_SMD:D_SOD-123
- D55: renamed from D53; footprint (none) -> Diode_SMD:D_SOD-123
- D56: renamed from D54; footprint (none) -> Diode_SMD:D_SOD-123
- D57: renamed from D55; footprint (none) -> Diode_SMD:D_SOD-123
- D58: renamed from D56; footprint (none) -> Diode_SMD:D_SOD-123
- D59: renamed from D57; footprint (none) -> Diode_SMD:D_SOD-123
- D6: renamed from D5; footprint (none) -> Diode_SMD:D_SOD-123
- D60: renamed from D58; footprint (none) -> Diode_SMD:D_SOD-123
- D61: renamed from D59; footprint (none) -> Diode_SMD:D_SOD-123
- D62: renamed from D60; footprint (none) -> Diode_SMD:D_SOD-123
- D63: renamed from D61; footprint (none) -> Diode_SMD:D_SOD-123
- D64: renamed from D62; footprint (none) -> Diode_SMD:D_SOD-123
- D65: renamed from D63; footprint (none) -> Diode_SMD:D_SOD-123
- D66: renamed from D64; footprint (none) -> Diode_SMD:D_SOD-123
- D67: renamed from D65; footprint (none) -> Diode_SMD:D_SOD-123
- D68: renamed from D66; footprint (none) -> Diode_SMD:D_SOD-123
- D69: renamed from D67; footprint (none) -> Diode_SMD:D_SOD-123
- D7: renamed from D6; footprint (none) -> Diode_SMD:D_SOD-123
- D70: renamed from D68; footprint (none) -> Diode_SMD:D_SOD-123
- D71: renamed from D69; footprint (none) -> Diode_SMD:D_SOD-123
- D72: renamed from D70; footprint (none) -> Diode_SMD:D_SOD-123
- D73: renamed from D71; footprint (none) -> Diode_SMD:D_SOD-123
- D74: renamed from D72; footprint (none) -> Diode_SMD:D_SOD-123
- D75: renamed from D73; footprint (none) -> Diode_SMD:D_SOD-123
- D76: renamed from D74; footprint (none) -> Diode_SMD:D_SOD-123
- D77: renamed from D75; footprint (none) -> Diode_SMD:D_SOD-123
- D78: renamed from D76; footprint (none) -> Diode_SMD:D_SOD-123
- D79: renamed from D77; footprint (none) -> Diode_SMD:D_SOD-123
- D8: renamed from D7; footprint (none) -> Diode_SMD:D_SOD-123
- D80: renamed from D78; footprint (none) -> Diode_SMD:D_SOD-123
- D81: renamed from D79; footprint (none) -> Diode_SMD:D_SOD-123
- D82: renamed from D80; footprint (none) -> Diode_SMD:D_SOD-123
- D83: renamed from D81; footprint (none) -> Diode_SMD:D_SOD-123
- D84: renamed from D82; footprint (none) -> Diode_SMD:D_SOD-123
- D9: renamed from D8; footprint (none) -> Diode_SMD:D_SOD-123
- S1: renamed from S0; footprint (none) -> keyboard:MX-Hotswap-1U
- S10: renamed from S9; footprint (none) -> keyboard:MX-Hotswap-1U
- S11: renamed from S10; footprint (none) -> keyboard:MX-Hotswap-1U
- S12: renamed from S11; footprint (none) -> keyboard:MX-Hotswap-1U
- S13: renamed from S12; footprint (none) -> keyboard:MX-Hotswap-1U
- S14: renamed from S13; footprint (none) -> keyboard:MX-Hotswap-1U
- S15: renamed from S14; footprint (none) -> keyboard:MX-Hotswap-1U
- S17: renamed from S15; footprint (none) -> keyboard:MX-Hotswap-1U
- S18: renamed from S16; footprint (none) -> keyboard:MX-Hotswap-1U
- S19: renamed from S17; footprint (none) -> keyboard:MX-Hotswap-1U
- S2: renamed from S1; footprint (none) -> keyboard:MX-Hotswap-1U
- S20: renamed from S18; footprint (none) -> keyboard:MX-Hotswap-1U
- S21: renamed from S19; footprint (none) -> keyboard:MX-Hotswap-1U
- S22: renamed from S20; footprint (none) -> keyboard:MX-Hotswap-1U
- S23: renamed from S21; footprint (none) -> keyboard:MX-Hotswap-1U
- S24: renamed from S22; footprint (none) -> keyboard:MX-Hotswap-1U
- S25: renamed from S23; footprint (none) -> keyboard:MX-Hotswap-1U
- S26: renamed from S24; footprint (none) -> keyboard:MX-Hotswap-1U
- S27: renamed from S25; footprint (none) -> keyboard:MX-Hotswap-1U
- S28: renamed from S26; footprint (none) -> keyboard:MX-Hotswap-1U
- S29: renamed from S27; footprint (none) -> keyboard:MX-Hotswap-1U
- S3: renamed from S2; footprint (none) -> keyboard:MX-Hotswap-1U
- S30: renamed from S28; footprint (none) -> keyboard:MX-Hotswap-2U
- S31: renamed from S29; footprint (none) -> keyboard:MX-Hotswap-1U
- S32: renamed from S30; footprint (none) -> keyboard:MX-Hotswap-1.5U
- S33: renamed from S31; footprint (none) -> keyboard:MX-Hotswap-1U
- S34: renamed from S32; footprint (none) -> keyboard:MX-Hotswap-1U
- S35: renamed from S33; footprint (none) -> keyboard:MX-Hotswap-1U
- S36: renamed from S34; footprint (none) -> keyboard:MX-Hotswap-1U
- S37: renamed from S35; footprint (none) -> keyboard:MX-Hotswap-1U
- S38: renamed from S36; footprint (none) -> keyboard:MX-Hotswap-1U
- S39: renamed from S37; footprint (none) -> keyboard:MX-Hotswap-1U
- S4: renamed from S3; footprint (none) -> keyboard:MX-Hotswap-1U
- S40: renamed from S38; footprint (none) -> keyboard:MX-Hotswap-1U
- S41: renamed from S39; footprint (none) -> keyboard:MX-Hotswap-1U
- S42: renamed from S40; footprint (none) -> keyboard:MX-Hotswap-1U
- S43: renamed from S41; footprint (none) -> keyboard:MX-Hotswap-1U
- S44: renamed from S42; footprint (none) -> keyboard:MX-Hotswap-1U
- S45: renamed from S43; footprint (none) -> keyboard:MX-Hotswap-1.5U
- S46: renamed from S44; footprint (none) -> keyboard:MX-Hotswap-1U
- S47: renamed from S45; footprint (none) -> keyboard:MX-Hotswap-1.75U
- S48: renamed from S46; footprint (none) -> keyboard:MX-Hotswap-1U
- S49: renamed from S47; footprint (none) -> keyboard:MX-Hotswap-1U
- S5: renamed from S4; footprint (none) -> keyboard:MX-Hotswap-1U
- S50: renamed from S48; footprint (none) -> keyboard:MX-Hotswap-1U
- S51: renamed from S49; footprint (none) -> keyboard:MX-Hotswap-1U
- S52: renamed from S50; footprint (none) -> keyboard:MX-Hotswap-1U
- S53: renamed from S51; footprint (none) -> keyboard:MX-Hotswap-1U
- S54: renamed from S52; footprint (none) -> keyboard:MX-Hotswap-1U
- S55: renamed from S53; footprint (none) -> keyboard:MX-Hotswap-1U
- S56: renamed from S54; footprint (none) -> keyboard:MX-Hotswap-1U
- S57: renamed from S55; footprint (none) -> keyboard:MX-Hotswap-1U
- S58: renamed from S56; footprint (none) -> keyboard:MX-Hotswap-1U
- S59: renamed from S57; footprint (none) -> keyboard:MX-Hotswap-2.25U
- S6: renamed from S5; footprint (none) -> keyboard:MX-Hotswap-1U
- S60: renamed from S58; footprint (none) -> keyboard:MX-Hotswap-1U
- S61: renamed from S59; footprint (none) -> keyboard:MX-Hotswap-2.25U
- S62: renamed from S60; footprint (none) -> keyboard:MX-Hotswap-1U
- S63: renamed from S61; footprint (none) -> keyboard:MX-Hotswap-1U
- S64: renamed from S62; footprint (none) -> keyboard:MX-Hotswap-1U
- S65: renamed from S63; footprint (none) -> keyboard:MX-Hotswap-1U
- S66: renamed from S64; footprint (none) -> keyboard:MX-Hotswap-1U
- S67: renamed from S65; footprint (none) -> keyboard:MX-Hotswap-1U
- S68: renamed from S66; footprint (none) -> keyboard:MX-Hotswap-1U
- S69: renamed from S67; footprint (none) -> keyboard:MX-Hotswap-1U
- S7: renamed from S6; footprint (none) -> keyboard:MX-Hotswap-1U
- S70: renamed from S68; footprint (none) -> keyboard:MX-Hotswap-1U
- S71: renamed from S69; footprint (none) -> keyboard:MX-Hotswap-1U
- S72: renamed from S70; footprint (none) -> keyboard:MX-Hotswap-1.75U
- S73: renamed from S71; footprint (none) -> keyboard:MX-Hotswap-1U
- S74: renamed from S72; footprint (none) -> keyboard:MX-Hotswap-1U
- S75: renamed from S73; footprint (none) -> keyboard:MX-Hotswap-1.25U
- S76: renamed from S74; footprint (none) -> keyboard:MX-Hotswap-1.25U
- S77: renamed from S75; footprint (none) -> keyboard:MX-Hotswap-1.25U
- S78: renamed from S76; footprint (none) -> keyboard:MX-Hotswap-6.25U
- S79: renamed from S77; footprint (none) -> keyboard:MX-Hotswap-1U
- S8: renamed from S7; footprint (none) -> keyboard:MX-Hotswap-1U
- S80: renamed from S78; footprint (none) -> keyboard:MX-Hotswap-1U
- S81: renamed from S79; footprint (none) -> keyboard:MX-Hotswap-1U
- S82: renamed from S80; footprint (none) -> keyboard:MX-Hotswap-1U
- S83: renamed from S81; footprint (none) -> keyboard:MX-Hotswap-1U
- S84: renamed from S82; footprint (none) -> keyboard:MX-Hotswap-1U
- S9: renamed from S8; footprint (none) -> keyboard:MX-Hotswap-1U
- renumbered A0 to A1
Connections:
- net +3V3: now also R1.1, R2.1, U1.1 (VDD)
- net GND: now also U1.2 (GND)
- net Row 0: now also D16.1 (K)
- net SDA: now reaches A1.19 (GPIO14)
- net SDA: now also R1.2, U1.4 (SDA)
- net SCL: now reaches A1.20 (GPIO15)
- net SCL: now also R2.2, U1.3 (SCL)
- net Col 15: now reaches A1.34 (GPIO28_ADC2)
- net Col 15: now also S16.1
- new net: D16.2 (A), S16.2
- no-connect marks 6 -> 8
