File: keyboard.kicad_sch (KiCad schematic)
At the start: 111 parts, among them J1 USB_C_Receptacle_USB2.0_14P, SW1 SW_Push, U1 STM32F072C8Tx, U2 MCP1700x-330xxTT, U3 USBLC6-2P6

Commit message: first full version of pcb complete
Parts:
- removed H1, H10, H2, H3, H4, H5, H6, H7, H8, H9: MountingHole, MountingHole:MountingHole_2.2mm_M2, symbol Mechanical:MountingHole
- removed LED1, LED10, LED11, LED12, LED13, LED14, LED15, LED16, LED17, LED18, LED19, LED2, LED20, LED21, LED22, LED23, LED24, LED25, LED26, LED27, LED28, LED29, LED3, LED30, LED31, LED32, LED33, LED34, LED35, LED36, LED37, LED38, LED39, LED4, LED40, LED41, LED42, LED43, LED44, LED45, LED46, LED47, LED48, LED49, LED5, LED50, LED51, LED52, LED53, LED54, LED55, LED56, LED57, LED58, LED59, LED6, LED60, LED61, LED62, LED63, LED64, LED65, LED66, LED67, LED68, LED69, LED7, LED70, LED71, LED72, LED73, LED74, LED75, LED76, LED77, LED78, LED79, LED8, LED80, LED81, LED82, LED83, LED84, LED9: SK6812MINI-E, keyboard:LED_6028R, symbol various:SK6812MINI-E
- added C10, C11, C12, C13, C14, C15, C16, C17, C18, C19, C20, C21, C22, C23, C24, C25, C26, C27, C28, C29, C30, C31, C32, C33: 100n, Capacitor_SMD:C_0603_1608Metric, symbol Device:C
- added U4: SN74LV1T125DBV, Package_TO_SOT_SMD:SOT-23-5, symbol Logic_LevelTranslator:SN74LV1T125DBV
Connections:
- net +5V: now also C10.1, C11.1, C12.1, C13.1, C14.1, C15.1, C16.1, C17.1, C18.1, C19.1, C20.1, C21.1, C22.1, C23.1, C24.1, C25.1, C26.1, C27.1, C28.1, C29.1, C30.1, C31.1, C32.1, C33.1, U4.5 (VCC)
- net ARGB_DIN: now also U4.2 (A)
- net Col 0: now also U1.25 (PB12); no longer U1.28 (PB15)
- net Col 1: now also U1.26 (PB13); no longer U1.27 (PB14)
- net Col 10: now also U1.40 (PB4); no longer U1.41 (PB5)
- net Col 11: now also U1.41 (PB5); no longer U1.40 (PB4)
- net Col 12: now also U1.42 (PB6); no longer U1.39 (PB3)
- net Col 13: now also U1.13 (PA3); no longer U1.20 (PB2)
- net Col 14: now also U1.14 (PA4); no longer U1.19 (PB1), U1.30 (PA9)
- net Col 15: now also U1.12 (PA2); no longer U1.29 (PA8)
- net Col 2: now also U1.27 (PB14); no longer U1.26 (PB13)
- net Col 3: now also U1.28 (PB15); no longer U1.25 (PB12)
- net Col 4: now also U1.29 (PA8); no longer U1.22 (PB11)
- net Col 5: now also U1.30 (PA9); no longer U1.21 (PB10)
- net Col 6: now also U1.31 (PA10); no longer U1.46 (PB9)
- net Col 7: now also U1.37 (PA14); no longer U1.45 (PB8)
- net Col 8: now also U1.38 (PA15); no longer U1.43 (PB7)
- net Col 9: now also U1.39 (PB3); no longer U1.42 (PB6)
- net GND: now also C10.2, C11.2, C12.2, C13.2, C14.2, C15.2, C16.2, C17.2, C18.2, C19.2, C20.2, C21.2, C22.2, C23.2, C24.2, C25.2, C26.2, C27.2, C28.2, C29.2, C30.2, C31.2, C32.2, C33.2, U4.1 (~{OE}), U4.3 (GND)
- net Row 0: now also U1.17 (PA7); no longer U1.13 (PA3)
- net Row 1: now also U1.18 (PB0); no longer U1.14 (PA4)
- net Row 2: now also U1.19 (PB1); no longer U1.15 (PA5)
- net Row 3: now also U1.20 (PB2); no longer U1.16 (PA6)
- net Row 4: now also U1.43 (PB7); no longer U1.17 (PA7)
- net Row 5: now also U1.21 (PB10); no longer U1.18 (PB0)
- new net 5V_ARGB_DIN: U4.4 (Y)
- no-connect marks 3 -> 7
Other:
- added sheet ARGB LEDS (leds.kicad_sch)
- note added: "Decoupling Capacitors for RGB LEDS (1 per 5-7 LEDS)"
- moved on the sheet: C1, C2, C3, C4, C5, C6, C7, C8, C9, J1, R1, R2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

Commit message: pcb ready for review
Parts:
- J1: footprint keyboard:USB_C_Receptacle_HRO_TYPE-C-31-M-12 -> keyboard:GCT_USB4105-GF-A-120-niv; symbol Connector:USB_C_Receptacle_USB2.0_14P -> usbc:USB4105-GF-A-120; MANUFACTURER (none) -> Global Connector Technology; MAXIMUM_PACKAGE_HEIGHT (none) -> 3.31mm; PARTREV (none) -> B3; STANDARD (none) -> Manufacturer Recommendations
- renumbered R3 to R2, R2 to R3
Connections:
- net +5V: now also J1.A4_B9 (VBUS), J1.B4_A9 (VBUS__1); no longer J1.A4 (VBUS), J1.A9 (VBUS), J1.B4 (VBUS), J1.B9 (VBUS)
- net GND: now also J1.A1_B12 (GND), J1.B1_A12 (GND__1), J1.SH1 (SHELL_GND), J1.SH2 (SHELL_GND__1), J1.SH3 (SHELL_GND__2), J1.SH4 (SHELL_GND__3), R3.1; no longer J1.A1 (GND), J1.A12 (GND), J1.B1 (GND), J1.B12 (GND), J1.S1 (SHIELD), R3.2
- net USB_DN: now also J1.A7 (DN1), J1.B7 (DN2); no longer J1.A6 (D+), J1.B6 (D+)
- net USB_DP: now also J1.A6 (DP1), J1.B6 (DP2); no longer J1.A7 (D-), J1.B7 (D-)
- net at J1.A5 (CC1): now also R2.1; no longer R3.1
- net at J1.B5 (CC2): now also R3.2; no longer R2.1
- no-connect marks 7 -> 14
Other:
- moved on the sheet: C1, C2, C3, C4, C5, C6, R1, R2, R3, SW1, U3
