File: _autosave-keyboard.kicad_sch (KiCad schematic)
At the start: 111 parts, among them J1 USB_C_Receptacle_USB2.0_14P, SW1 SW_Push, U1 STM32F072C8Tx, U2 MCP1700x-330xxTT, U3 USBLC6-2P6

Commit message: placed components on pcb
Parts:
- LED1, LED10, LED11, LED12, LED13, LED14, LED15, LED16, LED17, LED18, LED19, LED2, LED20, LED21, LED22, LED23, LED24, LED25, LED26, LED27, LED28, LED29, LED3, LED30, LED31, LED32, LED33, LED34, LED35, LED36, LED37, LED38, LED39, LED4, LED40, LED41, LED42, LED43, LED44, LED45, LED46, LED47, LED48, LED49, LED5, LED50, LED51, LED52, LED53, LED54, LED55, LED56, LED57, LED58, LED59, LED6, LED60, LED61, LED62, LED63, LED64, LED65, LED66, LED67, LED68, LED69, LED7, LED70, LED71, LED72, LED73, LED74, LED75, LED76, LED77, LED78, LED79, LED8, LED80, LED81, LED82, LED83, LED84, LED9: footprint PCM_marbastlib-various:LED_6028R -> keyboard:LED_6028R
