File: keyboard.kicad_pcb (KiCad board)
At the start: 2 copper layers, 336.1 x 124.1 mm, 172 parts, among them U1 OLED96-636

Commit message: placed components on pcb
Parts:
- removed A1: RaspberryPi_Pico, Module:RaspberryPi_Pico_Common_SMD
- added C1: 4.7u, Capacitor_SMD:C_0603_1608Metric, B.Cu at (221.5, 177.6)
- added C2: 100n, Capacitor_SMD:C_0603_1608Metric, B.Cu at (214.0, 174.9)
- added C3: 100n, Capacitor_SMD:C_0603_1608Metric, B.Cu at (224.2, 165.1)
- added C4: 100n, Capacitor_SMD:C_0603_1608Metric, B.Cu at (208.8, 165.1)
- added C5: 100n, Capacitor_SMD:C_0603_1608Metric, B.Cu at (224.5, 168.6)
- added C6: 10n, Capacitor_SMD:C_0603_1608Metric, B.Cu at (219.5, 160.4)
- added C7: 100n, Capacitor_SMD:C_0603_1608Metric, B.Cu at (224.3, 167.1)
- added C8: 1u, Capacitor_SMD:C_0603_1608Metric, B.Cu at (236.2, 172.1)
- added C9: 1u, Capacitor_SMD:C_0603_1608Metric, B.Cu at (232.8, 166.1)
- added H1: MountingHole, MountingHole:MountingHole_2.2mm_M2, F.Cu at (851.5, 194.7)
- added H10: MountingHole, MountingHole:MountingHole_2.2mm_M2, F.Cu at (857.5, 218.5)
- added H2: MountingHole, MountingHole:MountingHole_2.2mm_M2, F.Cu at (851.5, 200.7)
- added H3: MountingHole, MountingHole:MountingHole_2.2mm_M2, F.Cu at (851.5, 206.6)
- added H4: MountingHole, MountingHole:MountingHole_2.2mm_M2, F.Cu at (851.5, 212.6)
- added H5: MountingHole, MountingHole:MountingHole_2.2mm_M2, F.Cu at (851.5, 218.5)
- added H6: MountingHole, MountingHole:MountingHole_2.2mm_M2, F.Cu at (857.5, 194.7)
- added H7: MountingHole, MountingHole:MountingHole_2.2mm_M2, F.Cu at (857.5, 200.7)
- added H8: MountingHole, MountingHole:MountingHole_2.2mm_M2, F.Cu at (857.5, 206.6)
- added H9: MountingHole, MountingHole:MountingHole_2.2mm_M2, F.Cu at (857.5, 212.6)
- added J1: USB_C_Receptacle_USB2.0_14P, keyboard:USB_C_Receptacle_HRO_TYPE-C-31-M-12, B.Cu at (182.0, 58.1)
- added LED1: SK6812MINI-E, keyboard:LED_6028R, B.Cu at (58.1, 65.2)
- added LED10: SK6812MINI-E, keyboard:LED_6028R, B.Cu at (229.5, 65.2)
- added LED11: SK6812MINI-E, keyboard:LED_6028R, B.Cu at (248.6, 65.2)
- added LED12: SK6812MINI-E, keyboard:LED_6028R, B.Cu at (267.6, 65.2)
- added LED13: SK6812MINI-E, keyboard:LED_6028R, B.Cu at (286.7, 65.2)
- added LED14: SK6812MINI-E, keyboard:LED_6028R, B.Cu at (305.7, 65.2)
- added LED15: SK6812MINI-E, keyboard:LED_6028R, B.Cu at (324.8, 65.2)
- added LED16: SK6812MINI-E, keyboard:LED_6028R, B.Cu at (343.8, 65.2)
- added LED17: SK6812MINI-E, keyboard:LED_6028R, B.Cu at (58.1, 89.0)
- added LED18: SK6812MINI-E, keyboard:LED_6028R, B.Cu at (77.1, 89.0)
- added LED19: SK6812MINI-E, keyboard:LED_6028R, B.Cu at (96.2, 89.0)
- added LED2: SK6812MINI-E, keyboard:LED_6028R, B.Cu at (77.1, 65.2)
- added LED20: SK6812MINI-E, keyboard:LED_6028R, B.Cu at (115.2, 89.0)
- added LED21: SK6812MINI-E, keyboard:LED_6028R, B.Cu at (134.3, 89.0)
- added LED22: SK6812MINI-E, keyboard:LED_6028R, B.Cu at (153.3, 89.0)
- added LED23: SK6812MINI-E, keyboard:LED_6028R, B.Cu at (172.4, 89.0)
- added LED24: SK6812MINI-E, keyboard:LED_6028R, B.Cu at (191.4, 89.0)
- added LED25: SK6812MINI-E, keyboard:LED_6028R, B.Cu at (210.5, 89.0)
- added LED26: SK6812MINI-E, keyboard:LED_6028R, B.Cu at (229.5, 89.0)
- added LED27: SK6812MINI-E, keyboard:LED_6028R, B.Cu at (248.6, 89.0)
- added LED28: SK6812MINI-E, keyboard:LED_6028R, B.Cu at (267.6, 89.0)
- added LED29: SK6812MINI-E, keyboard:LED_6028R, B.Cu at (286.7, 89.0)
- added LED3: SK6812MINI-E, keyboard:LED_6028R, B.Cu at (96.2, 65.2)
- added LED30: SK6812MINI-E, keyboard:LED_6028R, B.Cu at (315.2, 89.0)
- added LED31: SK6812MINI-E, keyboard:LED_6028R, B.Cu at (343.8, 89.0)
- added LED32: SK6812MINI-E, keyboard:LED_6028R, B.Cu at (62.8, 108.1)
- added LED33: SK6812MINI-E, keyboard:LED_6028R, B.Cu at (86.7, 108.1)
- added LED34: SK6812MINI-E, keyboard:LED_6028R, B.Cu at (105.7, 108.1)
- added LED35: SK6812MINI-E, keyboard:LED_6028R, B.Cu at (124.8, 108.1)
- added LED36: SK6812MINI-E, keyboard:LED_6028R, B.Cu at (143.8, 108.1)
- added LED37: SK6812MINI-E, keyboard:LED_6028R, B.Cu at (162.8, 108.1)
- added LED38: SK6812MINI-E, keyboard:LED_6028R, B.Cu at (181.9, 108.1)
- added LED39: SK6812MINI-E, keyboard:LED_6028R, B.Cu at (200.9, 108.1)
- added LED4: SK6812MINI-E, keyboard:LED_6028R, B.Cu at (115.2, 65.2)
- added LED40: SK6812MINI-E, keyboard:LED_6028R, B.Cu at (220.0, 108.1)
- added LED41: SK6812MINI-E, keyboard:LED_6028R, B.Cu at (239.1, 108.1)
- added LED42: SK6812MINI-E, keyboard:LED_6028R, B.Cu at (258.1, 108.1)
- added LED43: SK6812MINI-E, keyboard:LED_6028R, B.Cu at (277.1, 108.1)
- added LED44: SK6812MINI-E, keyboard:LED_6028R, B.Cu at (296.2, 108.1)
- added LED45: SK6812MINI-E, keyboard:LED_6028R, B.Cu at (320.0, 108.1)
- added LED46: SK6812MINI-E, keyboard:LED_6028R, B.Cu at (343.8, 108.1)
- added LED47: SK6812MINI-E, keyboard:LED_6028R, B.Cu at (65.2, 127.2)
- added LED48: SK6812MINI-E, keyboard:LED_6028R, B.Cu at (91.4, 127.2)
- added LED49: SK6812MINI-E, keyboard:LED_6028R, B.Cu at (110.5, 127.2)
- added LED5: SK6812MINI-E, keyboard:LED_6028R, B.Cu at (134.3, 65.2)
- added LED50: SK6812MINI-E, keyboard:LED_6028R, B.Cu at (129.5, 127.2)
- added LED51: SK6812MINI-E, keyboard:LED_6028R, B.Cu at (148.6, 127.2)
- added LED52: SK6812MINI-E, keyboard:LED_6028R, B.Cu at (167.6, 127.2)
- added LED53: SK6812MINI-E, keyboard:LED_6028R, B.Cu at (186.7, 127.2)
- added LED54: SK6812MINI-E, keyboard:LED_6028R, B.Cu at (205.7, 127.2)
- added LED55: SK6812MINI-E, keyboard:LED_6028R, B.Cu at (224.8, 127.2)
- added LED56: SK6812MINI-E, keyboard:LED_6028R, B.Cu at (243.8, 127.2)
- added LED57: SK6812MINI-E, keyboard:LED_6028R, B.Cu at (262.9, 127.2)
- added LED58: SK6812MINI-E, keyboard:LED_6028R, B.Cu at (281.9, 127.2)
- added LED59: SK6812MINI-E, keyboard:LED_6028R, B.Cu at (312.9, 127.2)
- added LED6: SK6812MINI-E, keyboard:LED_6028R, B.Cu at (153.3, 65.2)
- added LED60: SK6812MINI-E, keyboard:LED_6028R, B.Cu at (343.8, 127.2)
- added LED61: SK6812MINI-E, keyboard:LED_6028R, B.Cu at (70.0, 146.2)
- added LED62: SK6812MINI-E, keyboard:LED_6028R, B.Cu at (100.9, 146.2)
- added LED63: SK6812MINI-E, keyboard:LED_6028R, B.Cu at (120.0, 146.2)
- added LED64: SK6812MINI-E, keyboard:LED_6028R, B.Cu at (139.0, 146.2)
- added LED65: SK6812MINI-E, keyboard:LED_6028R, B.Cu at (158.1, 146.2)
- added LED66: SK6812MINI-E, keyboard:LED_6028R, B.Cu at (177.1, 146.2)
- added LED67: SK6812MINI-E, keyboard:LED_6028R, B.Cu at (196.2, 146.2)
- added LED68: SK6812MINI-E, keyboard:LED_6028R, B.Cu at (215.2, 146.2)
- added LED69: SK6812MINI-E, keyboard:LED_6028R, B.Cu at (234.3, 146.2)
- added LED7: SK6812MINI-E, keyboard:LED_6028R, B.Cu at (172.4, 65.2)
- added LED70: SK6812MINI-E, keyboard:LED_6028R, B.Cu at (253.3, 146.2)
- added LED71: SK6812MINI-E, keyboard:LED_6028R, B.Cu at (272.4, 146.2)
- added LED72: SK6812MINI-E, keyboard:LED_6028R, B.Cu at (298.6, 146.2)
- added LED73: SK6812MINI-E, keyboard:LED_6028R, B.Cu at (324.8, 146.2)
- added LED74: SK6812MINI-E, keyboard:LED_6028R, B.Cu at (343.8, 146.2)
- added LED75: SK6812MINI-E, keyboard:LED_6028R, B.Cu at (60.5, 165.2)
- added LED76: SK6812MINI-E, keyboard:LED_6028R, B.Cu at (84.3, 165.2)
- added LED77: SK6812MINI-E, keyboard:LED_6028R, B.Cu at (108.1, 165.2)
- added LED78: SK6812MINI-E, keyboard:LED_6028R, B.Cu at (179.5, 165.2)
- added LED79: SK6812MINI-E, keyboard:LED_6028R, B.Cu at (248.6, 165.2)
- added LED8: SK6812MINI-E, keyboard:LED_6028R, B.Cu at (191.4, 65.2)
- added LED80: SK6812MINI-E, keyboard:LED_6028R, B.Cu at (267.6, 165.2)
- added LED81: SK6812MINI-E, keyboard:LED_6028R, B.Cu at (286.7, 165.2)
- added LED82: SK6812MINI-E, keyboard:LED_6028R, B.Cu at (305.7, 165.2)
- added LED83: SK6812MINI-E, keyboard:LED_6028R, B.Cu at (324.8, 165.2)
- added LED84: SK6812MINI-E, keyboard:LED_6028R, B.Cu at (343.8, 165.2)
- added LED9: SK6812MINI-E, keyboard:LED_6028R, B.Cu at (210.5, 65.2)
- added R3: 5.1k, Resistor_SMD:R_0603_1608Metric, B.Cu at (185.0, 64.1)
- added SW1: SW_Push, Button_Switch_SMD:SW_Push_1P1T_NO_CK_KMR2, B.Cu at (203.0, 163.9)
- added U2: MCP1700x-330xxTT, Package_TO_SOT_SMD:SOT-23, B.Cu at (233.9, 169.1)
- added U3: USBLC6-2P6, Package_TO_SOT_SMD:SOT-666, B.Cu at (182.0, 78.6)
- R1: value 4.7k -> 10k
- R2: value 4.7k -> 5.1k
- U1: value OLED96-636 -> STM32F072C8Tx; footprint keyboard:MODULE_DM-OLED096-636 -> Package_QFP:LQFP-48_7x7mm_P0.5mm; moved to B.Cu
- moved R2 167.5 mm to (179.5, 64.1)
- moved R1 159.3 mm to (211.0, 160.1), turned to 180 degrees
- moved U1 135.8 mm to (216.5, 167.6), turned to 180 degrees
- moved D56 38.4 mm to (236.6, 131.2)
- moved D60 38.4 mm to (336.6, 131.2)
- moved D12 38.4 mm to (260.4, 69.2)
- moved D13 38.4 mm to (279.5, 69.2)
- moved D16 38.4 mm to (336.6, 69.2)
- moved D23 38.4 mm to (165.2, 93.0)
- moved D28 38.4 mm to (260.4, 93.0)
- moved D29 38.4 mm to (279.5, 93.0)
- moved D30 38.4 mm to (308.1, 93.0)
- moved D31 38.4 mm to (336.6, 93.0)
- moved D51 38.4 mm to (141.4, 131.2)
- moved D7 38.4 mm to (165.2, 69.2)
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Connections:
- R1 pad 1: +3V3 -> /BOOT0
- R1 pad 2: /SDA -> GND
- R2 pad 1: +3V3 -> Net-(J1-CC1)
- R2 pad 2: /SCL -> GND
- U1 pad 2: GND -> unconnected-(U1-PC13-Pad2)
- U1 pad 3: /SCL -> unconnected-(U1-PC14-Pad3)
- U1 pad 4: /SDA -> unconnected-(U1-PC15-Pad4)
Routing:
- net Col 0: track 425.0 -> 0.00 mm, vias 13 -> 0
- net Row 5: track 415.3 -> 0.00 mm, vias 2 -> 0
- net Col 1: track 399.6 -> 0.00 mm, vias 13 -> 0
- net Row 4: track 390.1 -> 0.00 mm, vias 2 -> 0
- net Row 3: track 389.5 -> 0.00 mm, vias 6 -> 0
- net Col 2: track 387.8 -> 0.00 mm, vias 13 -> 0
- net Row 2: track 367.2 -> 0.00 mm, vias 2 -> 0
- net Row 1: track 356.9 -> 0.00 mm, vias 2 -> 0
- net Col 5: track 347.1 -> 0.00 mm, vias 13 -> 0
- net Col 3: track 339.9 -> 0.00 mm, vias 11 -> 0
- net Col 4: track 337.4 -> 0.00 mm, vias 11 -> 0
- net Row 0: track 336.3 -> 0.00 mm
- net Col 7: track 294.9 -> 0.00 mm, vias 11 -> 0
- net Col 9: track 284.4 -> 0.00 mm, vias 13 -> 0
- net Col 8: track 283.7 -> 0.00 mm, vias 11 -> 0
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- removed copper zone on B.Cu, net GND
Other:
- board size 336.1 x 124.1 mm -> 309.9 x 124.2 mm
