File: matrix.kicad_sch (KiCad schematic)
At the start: 168 parts

Commit message: first full version of pcb complete
Changed lines of the file:
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@@
 	(generator "eeschema")
 	(generator_version "9.0")
-	(paper "A3")
+	(paper "A4")
 	(junction
 		(at 55.88 77.47)
@@
 	(wire
 		(pts
-			(xy 167.64 189.23) (xy 177.8 189.23)
+			(xy 167.64 189.23) (xy 168.91 189.23)
 		)
 		(stroke
@@
 	(global_label "Row 5"
 		(shape input)
-		(at 177.8 189.23 0)
+		(at 168.91 189.23 0)
 		(fields_autoplaced yes)
 		(effects
@@
 		)
 		(property "Intersheetrefs" "${INTERSHEET_REFS}"
-			(at 186.7118 189.23 0)
+			(at 177.8218 189.23 0)
 			(effects
 				(font
